File: Hardware/EAGLE/AS6212_breakout.brd (EAGLE design)
At the start: 25.4 x 25.4 mm, 19 parts, among them J2 QWIIC_RIGHT_ANGLE, J3 QWIIC_RIGHT_ANGLE, U1 AS6212

Commit message: v01 main push
Updated Eagle files and source software
Parts:
- moved U1 3.81 mm to (12.7, 16.5), turned to 180 degrees
- moved JP5 3.23 mm to (22.5, 4.52), turned to 90 degrees
- moved JP4 2.54 mm to (10.2, 5.08)
- moved JP6 2.54 mm to (7.58, 5.00)
- moved R1 1.80 mm to (21.3, 3.23), turned to 0 degrees
- moved R2 1.80 mm to (21.2, 5.77), turned to 0 degrees
- moved C1 0.60 mm to (7.62, 8.89), turned to 90 degrees
Connections:
- net ADD1: now also J1.1; no longer J1.2
- net GND: now also J1.2; no longer J1.1
Routing:
- net VCC: track 69.4 -> 50.0 mm, vias 3 -> 1
- net SCL: track 39.9 -> 59.2 mm, vias 5 -> 2
- net ADD1: track 17.8 -> 31.3 mm, vias 2 -> 1
- net SDA: track 41.3 -> 49.1 mm, vias 0 -> 2
- net ADD0: track 25.9 -> 19.4 mm, vias 3 -> 1
- net N$2: track 2.20 -> 0.00 mm, vias 1 -> 0
- net N$1: track 2.20 -> 0.00 mm, vias 1 -> 0
- net GND: track 2.00 -> 2.22 mm, vias 4 -> 1
Other:
- outline, holes or cut-outs redrawn

Commit message: Rev 02 push
First production version of breakout board - push ready
Parts:
- R3: value 330 -> 10k
Routing:
- net VCC: track 50.0 -> 54.8 mm, vias 1 -> 2
- net N$2: track 0.00 -> 3.82 mm, vias 0 -> 1
- net N$1: track 0.00 -> 2.81 mm, vias 0 -> 1
- net SCL: track 59.2 -> 61.7 mm
- net GND: vias 1 -> 10
Other:
- board text added: "B"
- board text added: "W"
Changed lines of the file:
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@@
 <wire x1="7.62" y1="17.78" x2="8.89" y2="17.78" width="0.1524" layer="20" curve="-180"/>
 <wire x1="16.51" y1="17.78" x2="17.78" y2="17.78" width="0.1524" layer="20" curve="-180"/>
+<text x="1.905" y="19.05" size="1.016" layer="21" font="vector" ratio="20">B</text>
+<text x="2.3114" y="18.288" size="1.016" layer="21" font="vector" ratio="20">W</text>
 </plain>
 <attributes>
@@
 <attribute name="VALUE" x="3.1115" y="2.8575" size="0.6096" layer="27" font="vector" ratio="20" align="top-center"/>
 </element>
-<element name="R3" library="SparkFun-Resistors" package="0603" value="330" x="3.175" y="6.5405" smashed="yes">
-<attribute name="PROD_ID" value="RES-00818" x="3.175" y="6.5405" size="1.778" layer="27" display="off"/>
-<attribute name="VALUE" x="3.1115" y="8.001" size="0.6096" layer="27" font="vector" ratio="20" align="top-center"/>
+<element name="R3" library="SparkFun-Resistors" package="0603" value="10k" x="3.175" y="6.5405" smashed="yes">
+<attribute name="PROD_ID" value="RES-00824" x="3.175" y="6.5405" size="1.778" layer="27" display="off"/>
+<attribute name="VALUE" value="10k" x="3.1115" y="8.001" size="0.6096" layer="27" font="vector" ratio="20" align="top-center"/>
 </element>
 <element name="JP7" library="SparkFun-Jumpers" package="SMT-JUMPER_2_NC_TRACE_SILK" package3d_urn="urn:adsk.eagle:package:39281/1" value="JUMPER-SMT_2_NC_TRACE_SILK" x="3.1115" y="5.1435" smashed="yes" rot="MR180"/>
@@
 <wire x1="7.755" y1="13.2" x2="5.08" y2="13.2" width="0.254" layer="1"/>
 <wire x1="8.755" y1="12.2" x2="7.755" y2="13.2" width="0.254" layer="1"/>
-<wire x1="17.78" y1="12.2" x2="17.78" y2="1.27" width="0.254" layer="1"/>
+<wire x1="17.78" y1="12.2" x2="17.78" y2="4.445" width="0.254" layer="1"/>
+<wire x1="17.78" y1="4.445" x2="17.78" y2="1.27" width="0.254" layer="1"/>
 <wire x1="4.025" y1="6.5405" x2="4.8895" y2="6.5405" width="0.254" layer="1"/>
 <wire x1="5.8185" y1="5.6115" x2="7.62" y2="5.6115" width="0.254" layer="1"/>
@@
 <wire x1="3.81" y1="12.7" x2="3.81" y2="9.525" width="0.254" layer="1"/>
 <wire x1="3.81" y1="9.525" x2="5.345" y2="7.99" width="0.254" layer="1"/>
-<wire x1="17.78" y1="4.6736" x2="22.5044" y2="4.5212" width="0" layer="19" extent="16-16"/>
+<wire x1="17.78" y1="4.445" x2="17.835" y2="4.5" width="0.254" layer="1"/>
+<wire x1="17.835" y1="4.5" x2="20.32" y2="4.5" width="0.254" layer="1"/>
+<via x="20.32" y="4.5" extent="1-16" drill="0.508"/>
+<wire x1="20.32" y1="4.5" x2="22.4832" y2="4.5" width="0.254" layer="16"/>
+<wire x1="22.4832" y1="4.5" x2="22.5044" y2="4.5212" width="0.254" layer="16"/>
 </signal>
 <signal name="ADD0">
@@
 <wire x1="16.2814" y1="14.1986" x2="15.875" y2="14.605" width="0.254" layer="1"/>
 <wire x1="12.7" y1="4.6736" x2="12.7" y2="1.27" width="0.254" layer="16"/>
-<wire x1="20.42" y1="3.23" x2="20.42" y2="2.44" width="0.254" layer="1"/>
-<wire x1="20.42" y1="2.44" x2="20.955" y2="1.905" width="0.254" layer="1"/>
-<wire x1="23.495" y1="1.905" x2="24.13" y2="2.54" width="0.254" layer="1"/>
-<wire x1="24.13" y1="2.54" x2="24.13" y2="7.62" width="0.254" layer="1"/>
+<wire x1="20.42" y1="3.23" x2="20.42" y2="1.17" width="0.254" layer="1"/>
+<wire x1="20.42" y1="1.17" x2="20.955" y2="0.635" width="0.254" layer="1"/>
+<wire x1="23.495" y1="0.635" x2="24.13" y2="1.27" width="0.254" layer="1"/>
+<wire x1="24.13" y1="1.27" x2="24.13" y2="7.62" width="0.254" layer="1"/>
 <wire x1="24.13" y1="7.62" x2="23.495" y2="8.255" width="0.254" layer="1"/>
 <wire x1="23.495" y1="8.255" x2="22.86" y2="8.255" width="0.254" layer="1"/>
@@
 <wire x1="22.225" y1="13.335" x2="21.36" y2="14.2" width="0.254" layer="1"/>
 <wire x1="21.36" y1="14.2" x2="20.32" y2="14.2" width="0.254" layer="1"/>
-<wire x1="20.955" y1="1.905" x2="23.495" y2="1.905" width="0.254" layer="1"/>
+<wire x1="20.955" y1="0.635" x2="23.495" y2="0.635" width="0.254" layer="1"/>
 <wire x1="12.7" y1="8.89" x2="10.795" y2="10.795" width="0.254" layer="1"/>
 <wire x1="5.485" y1="10.795" x2="5.08" y2="11.2" width="0.254" layer="1"/>
@@
 <wire x1="11.43" y1="16.51" x2="10.16" y2="16.51" width="0.254" layer="1"/>
 <via x="10.16" y="16.51" extent="1-16" drill="0.508"/>
+<via x="15.24" y="19.05" extent="1-16" drill="0.508"/>
+<via x="19.05" y="10.16" extent="1-16" drill="0.508"/>
+<via x="10.16" y="17.78" extent="1-16" drill="0.508"/>
+<via x="10.16" y="15.24" extent="1-16" drill="0.508"/>
+<via x="13.97" y="19.05" extent="1-16" drill="0.508"/>
+<via x="15.24" y="20.32" extent="1-16" drill="0.508"/>
+<via x="13.97" y="20.32" extent="1-16" drill="0.508"/>
+<via x="13.97" y="17.78" extent="1-16" drill="0.508"/>
+<via x="15.24" y="17.78" extent="1-16" drill="0.508"/>
 </signal>
 <signal name="ADD1">
@@
 <contactref element="JP5" pad="3"/>
 <contactref element="R2" pad="2"/>
-<wire x1="22.08" y1="5.77" x2="22.5044" y2="5.5626" width="0" layer="19" extent="1-16"/>
+<wire x1="22.5044" y1="5.5626" x2="22.225" y2="5.842" width="0.254" layer="16"/>
+<wire x1="22.225" y1="5.842" x2="22.225" y2="6.985" width="0.254" layer="16"/>
+<via x="22.225" y="6.985" extent="1-16" drill="0.508"/>
+<wire x1="22.225" y1="6.985" x2="22.225" y2="5.915" width="0.254" layer="1"/>
+<wire x1="22.225" y1="5.915" x2="22.08" y2="5.77" width="0.254" layer="1"/>
 </signal>
 <signal name="N$2">
 <contactref element="JP5" pad="1"/>
 <contactref element="R1" pad="2"/>
-<wire x1="22.12" y1="3.23" x2="22.5044" y2="3.4798" width="0" layer="19" extent="1-16"/>
+<wire x1="22.12" y1="3.23" x2="22.225" y2="3.125" width="0.254" layer="1"/>
+<wire x1="22.225" y1="3.125" x2="22.225" y2="1.524" width="0.254" layer="1"/>
+<via x="22.225" y="1.524" extent="1-16" drill="0.508"/>
+<wire x1="22.5044" y1="1.8034" x2="22.225" y2="1.524" width="0.254" layer="16"/>
+<wire x1="22.5044" y1="3.4798" x2="22.5044" y2="1.8034" width="0.254" layer="16"/>
 </signal>
 <signal name="N$3">
@@
 <mfgpreviewcolor name="substratecolor" color="0xFF786E46"/>
 </mfgpreviewcolors>
+<errors>
+</errors>
 </board>
 </drawing>

Commit message: Configuration register updates
small changes to software and hardware.
Parts:
- R3: value 10k -> 1k
Changed lines of the file:
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@@
 <drawing>
 <settings>
-<setting alwaysvectorfont="yes"/>
+<setting alwaysvectorfont="no"/>
 <setting verticaltext="up"/>
 </settings>
@@
 <attribute name="VALUE" x="3.1115" y="2.8575" size="0.6096" layer="27" font="vector" ratio="20" align="top-center"/>
 </element>
-<element name="R3" library="SparkFun-Resistors" package="0603" value="10k" x="3.175" y="6.5405" smashed="yes">
-<attribute name="PROD_ID" value="RES-00824" x="3.175" y="6.5405" size="1.778" layer="27" display="off"/>
-<attribute name="VALUE" value="10k" x="3.1115" y="8.001" size="0.6096" layer="27" font="vector" ratio="20" align="top-center"/>
+<element name="R3" library="SparkFun-Resistors" package="0603" value="1k" x="3.175" y="6.5405" smashed="yes">
+<attribute name="PROD_ID" value="RES-07856" x="3.175" y="6.5405" size="1.778" layer="27" display="off"/>
+<attribute name="VALUE" value="1k" x="3.1115" y="8.001" size="0.6096" layer="27" font="vector" ratio="20" align="top-center"/>
 </element>
 <element name="JP7" library="SparkFun-Jumpers" package="SMT-JUMPER_2_NC_TRACE_SILK" package3d_urn="urn:adsk.eagle:package:39281/1" value="JUMPER-SMT_2_NC_TRACE_SILK" x="3.1115" y="5.1435" smashed="yes" rot="MR180"/>
