File: Hardware/EAGLE/AS6212_breakout.brd (EAGLE design)
At the start: 25.4 x 25.4 mm, 19 parts, among them J2 QWIIC_RIGHT_ANGLE, J3 QWIIC_RIGHT_ANGLE, U1 AS6212

Commit message: Board design rework & datasheet upload
Parts:
- added FD1, FD2: FIDUCIAL0.2MM, SparkFun-Aesthetics:FIDUCIAL-0.2MM
- added U$1: (no value), SparkFun-Aesthetics:QWIIC_5.5MM
- moved JP6 10.2 mm to (17.7, 5.00)
- moved C1 9.25 mm to (5.08, 17.8), turned to 0 degrees
- moved JP3 7.62 mm to (10.2, 5.08)
- moved U1 3.81 mm to (12.7, 12.7), turned to 0 degrees
- moved R1 3.44 mm to (21.3, 6.67), turned to 270 degrees
- moved R2 2.74 mm to (23.8, 6.71), turned to 270 degrees
- moved JP1 2.54 mm to (12.7, 5.08)
- moved JP2 2.54 mm to (15.2, 5.08)
- moved JP4 2.54 mm to (7.62, 5.08)
- moved JP5 0.92 mm to (22.6, 5.44), turned to 180 degrees
- turned R3 to 180 degrees
Connections:
- net ADD1: now also J1.5; no longer J1.1
- net GND: now also J1.1; no longer J1.2
- net SCL: now also J1.4; no longer J1.3
- net SDA: now also J1.3; no longer J1.4
- net VCC: now also J1.2; no longer J1.5
Routing:
- net SCL: track 61.7 -> 41.8 mm
- net ADD1: track 31.3 -> 14.7 mm
- net VCC: track 54.8 -> 65.3 mm, vias 2 -> 3
- net SDA: track 49.1 -> 53.7 mm
- net GND: track 2.22 -> 0.00 mm, vias 10 -> 7
- net N$4: track 1.64 -> 3.59 mm
- net N$2: track 3.82 -> 4.98 mm
- net N$3: track 2.84 -> 3.88 mm
- net N$1: track 2.81 -> 3.51 mm
Other:
- outline, holes or cut-outs redrawn
